File: Hardware/LilyPad_LED_5pcs.sch (EAGLE design)
At the start: 21 parts

Commit message: Updated files
Parts:
- added LOGO1: SFE_LOGO_NAME_FLAME.1_INCH, SparkFun-Aesthetics:SFE_LOGO_NAME_FLAME.1_INCH
- added LOGO2: OSHW-LOGOL, SparkFun-Aesthetics:OSHW-LOGOL
- added U$1: REVISION, SparkFun-Aesthetics:REVISION
Changed lines of the file:
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@@
 <part name="ST10" library="LilyPad-Wearables" deviceset="SEWTAP" device="6"/>
 <part name="FRAME1" library="SparkFun-Aesthetics" deviceset="FRAME-LETTER" device=""/>
+<part name="LOGO1" library="SparkFun-Aesthetics" deviceset="SFE_LOGO_NAME_FLAME" device=".1_INCH"/>
+<part name="LOGO2" library="SparkFun-Aesthetics" deviceset="OSHW-LOGO" device="L"/>
+<part name="U$1" library="SparkFun-Aesthetics" deviceset="REVISION" device=""/>
 </parts>
 <sheets>
 <sheet>
 <plain>
-<text x="165.862" y="7.874" size="2.54" layer="94">Mary West</text>
+<text x="168.402" y="6.604" size="2.54" layer="94">Mary West</text>
 <text x="236.22" y="7.62" size="2.54" layer="94">V02</text>
 <text x="165.608" y="11.43" size="2.54" layer="94">Leah Beuchley</text>
@@
 <instance part="FRAME1" gate="G$1" x="0" y="0"/>
 <instance part="FRAME1" gate="V" x="147.32" y="0"/>
+<instance part="LOGO1" gate="G$1" x="165.1" y="35.56"/>
+<instance part="LOGO2" gate="G$1" x="233.68" y="48.26"/>
+<instance part="U$1" gate="G$1" x="148.59" y="7.112"/>
 </instances>
 <busses>

Commit message: updated brd and sch files
Parts:
- removed LOGO1: SFE_LOGO_NAME_FLAME.1_INCH, SparkFun-Aesthetics:SFE_LOGO_NAME_FLAME.1_INCH
- removed LOGO2: OSHW-LOGOL, SparkFun-Aesthetics:OSHW-LOGOL
- removed U$1: REVISION, SparkFun-Aesthetics:REVISION
- added U$6: REVISION, SparkFun-Aesthetics:REVISION
- renumbered ST1 to LED+1, ST10 to LED-5, ST2 to LED-1, ST3 to LED+2, ST4 to LED-2, ST5 to LED+3, ST6 to LED-3, ST7 to LED+4, ST8 to LED-4, ST9 to LED+5
Connections:
- net N$1 renamed 3
- net N$10 renamed 12
- net N$11 renamed 11
- net N$12 renamed 10
- net N$13 renamed 13
- net N$14 renamed 14
- net N$15 renamed 15
- net N$2 renamed 1
- net N$3 renamed 2
- net N$4 renamed 4
- net N$5 renamed 5
- net N$6 renamed 6
- net N$7 renamed 7
- net N$8 renamed 8
- net N$9 renamed 9
Other:
- note added: "L. Buechley"
- note added: "M. West"
- note added: "v02"
- note removed: "Leah Beuchley"
- note removed: "Mary West"
- note removed: "V02"
Changed lines of the file:
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@@
 <part name="R4" library="SparkFun-Resistors" deviceset="150OHM-1/10W-1%(0603)" device="" value="150"/>
 <part name="R5" library="SparkFun-Resistors" deviceset="150OHM-1/10W-1%(0603)" device="" value="150"/>
-<part name="ST1" library="LilyPad-Wearables" deviceset="SEWTAP" device="6"/>
-<part name="ST2" library="LilyPad-Wearables" deviceset="SEWTAP" device="6"/>
-<part name="ST3" library="LilyPad-Wearables" deviceset="SEWTAP" device="6"/>
-<part name="ST4" library="LilyPad-Wearables" deviceset="SEWTAP" device="6"/>
-<part name="ST5" library="LilyPad-Wearables" deviceset="SEWTAP" device="6"/>
-<part name="ST6" library="LilyPad-Wearables" deviceset="SEWTAP" device="6"/>
-<part name="ST7" library="LilyPad-Wearables" deviceset="SEWTAP" device="6"/>
-<part name="ST8" library="LilyPad-Wearables" deviceset="SEWTAP" device="6"/>
-<part name="ST9" library="LilyPad-Wearables" deviceset="SEWTAP" device="6"/>
-<part name="ST10" library="LilyPad-Wearables" deviceset="SEWTAP" device="6"/>
+<part name="LED+1" library="LilyPad-Wearables" deviceset="SEWTAP" device="6"/>
+<part name="LED-1" library="LilyPad-Wearables" deviceset="SEWTAP" device="6"/>
+<part name="LED+2" library="LilyPad-Wearables" deviceset="SEWTAP" device="6"/>
+<part name="LED-2" library="LilyPad-Wearables" deviceset="SEWTAP" device="6"/>
+<part name="LED+3" library="LilyPad-Wearables" deviceset="SEWTAP" device="6"/>
+<part name="LED-3" library="LilyPad-Wearables" deviceset="SEWTAP" device="6"/>
+<part name="LED+4" library="LilyPad-Wearables" deviceset="SEWTAP" device="6"/>
+<part name="LED-4" library="LilyPad-Wearables" deviceset="SEWTAP" device="6"/>
+<part name="LED+5" library="LilyPad-Wearables" deviceset="SEWTAP" device="6"/>
+<part name="LED-5" library="LilyPad-Wearables" deviceset="SEWTAP" device="6"/>
 <part name="FRAME1" library="SparkFun-Aesthetics" deviceset="FRAME-LETTER" device=""/>
-<part name="LOGO1" library="SparkFun-Aesthetics" deviceset="SFE_LOGO_NAME_FLAME" device=".1_INCH"/>
-<part name="LOGO2" library="SparkFun-Aesthetics" deviceset="OSHW-LOGO" device="L"/>
-<part name="U$1" library="SparkFun-Aesthetics" deviceset="REVISION" device=""/>
+<part name="U$6" library="SparkFun-Aesthetics" deviceset="REVISION" device=""/>
 </parts>
 <sheets>
 <sheet>
 <plain>
-<text x="168.402" y="6.604" size="2.54" layer="94">Mary West</text>
-<text x="236.22" y="7.62" size="2.54" layer="94">V02</text>
-<text x="165.608" y="11.43" size="2.54" layer="94">Leah Beuchley</text>
+<text x="168.402" y="6.604" size="2.54" layer="94">M. West</text>
+<text x="166.116" y="11.43" size="2.54" layer="94">L. Buechley</text>
+<text x="238.76" y="7.62" size="1.778" layer="94">v02</text>
 </plain>
 <instances>
@@
 <instance part="R4" gate="G$1" x="101.6" y="81.28" rot="R180"/>
 <instance part="R5" gate="G$1" x="101.6" y="66.04" rot="R180"/>
-<instance part="ST1" gate="G$1" x="68.58" y="127" rot="R180"/>
-<instance part="ST2" gate="G$1" x="121.92" y="127"/>
-<instance part="ST3" gate="G$1" x="68.58" y="111.76" rot="R180"/>
-<instance part="ST4" gate="G$1" x="121.92" y="111.76"/>
-<instance part="ST5" gate="G$1" x="68.58" y="96.52" rot="R180"/>
-<instance part="ST6" gate="G$1" x="121.92" y="96.52"/>
-<instance part="ST7" gate="G$1" x="68.58" y="81.28" rot="R180"/>
-<instance part="ST8" gate="G$1" x="121.92" y="81.28"/>
-<instance part="ST9" gate="G$1" x="68.58" y="66.04" rot="R180"/>
-<instance part="ST10" gate="G$1" x="121.92" y="66.04"/>
+<instance part="LED+1" gate="G$1" x="68.58" y="127" rot="R180"/>
+<instance part="LED-1" gate="G$1" x="121.92" y="127"/>
+<instance part="LED+2" gate="G$1" x="68.58" y="111.76" rot="R180"/>
+<instance part="LED-2" gate="G$1" x="121.92" y="111.76"/>
+<instance part="LED+3" gate="G$1" x="68.58" y="96.52" rot="R180"/>
+<instance part="LED-3" gate="G$1" x="121.92" y="96.52"/>
+<instance part="LED+4" gate="G$1" x="68.58" y="81.28" rot="R180"/>
+<instance part="LED-4" gate="G$1" x="121.92" y="81.28"/>
+<instance part="LED+5" gate="G$1" x="68.58" y="66.04" rot="R180"/>
+<instance part="LED-5" gate="G$1" x="121.92" y="66.04"/>
 <instance part="FRAME1" gate="G$1" x="0" y="0"/>
 <instance part="FRAME1" gate="V" x="147.32" y="0"/>
-<instance part="LOGO1" gate="G$1" x="165.1" y="35.56"/>
-<instance part="LOGO2" gate="G$1" x="233.68" y="48.26"/>
-<instance part="U$1" gate="G$1" x="148.59" y="7.112"/>
+<instance part="U$6" gate="G$1" x="148.59" y="6.604"/>
 </instances>
 <busses>
 </busses>
 <nets>
-<net name="N$1" class="0">
+<net name="3" class="0">
 <segment>
 <pinref part="R1" gate="G$1" pin="1"/>
-<pinref part="ST2" gate="G$1" pin="1"/>
+<pinref part="LED-1" gate="G$1" pin="1"/>
 <wire x1="106.68" y1="127" x2="119.38" y2="127" width="0.1524" layer="91"/>
 </segment>
 </net>
-<net name="N$2" class="0">
+<net name="1" class="0">
 <segment>
-<pinref part="ST1" gate="G$1" pin="1"/>
+<pinref part="LED+1" gate="G$1" pin="1"/>
 <pinref part="D1" gate="G$1" pin="A"/>
 <wire x1="71.12" y1="127" x2="83.82" y2="127" width="0.1524" layer="91"/>
 </segment>
 </net>
-<net name="N$3" class="0">
+<net name="2" class="0">
 <segment>
 <pinref part="D1" gate="G$1" pin="C"/>
@@
 </segment>
 </net>
-<net name="N$4" class="0">
+<net name="4" class="0">
 <segment>
-<pinref part="ST3" gate="G$1" pin="1"/>
+<pinref part="LED+2" gate="G$1" pin="1"/>
 <pinref part="D2" gate="G$1" pin="A"/>
 <wire x1="71.12" y1="111.76" x2="83.82" y2="111.76" width="0.1524" layer="91"/>
 </segment>
 </net>
-<net name="N$5" class="0">
+<net name="5" class="0">
 <segment>
 <pinref part="D2" gate="G$1" pin="C"/>
@@
 </segment>
 </net>
-<net name="N$6" class="0">
+<net name="6" class="0">
 <segment>
 <pinref part="R2" gate="G$1" pin="1"/>
-<pinref part="ST4" gate="G$1" pin="1"/>
+<pinref part="LED-2" gate="G$1" pin="1"/>
 <wire x1="106.68" y1="111.76" x2="119.38" y2="111.76" width="0.1524" layer="91"/>
 </segment>
 </net>
-<net name="N$7" class="0">
+<net name="7" class="0">
 <segment>
-<pinref part="ST5" gate="G$1" pin="1"/>
+<pinref part="LED+3" gate="G$1" pin="1"/>
 <pinref part="D3" gate="G$1" pin="A"/>
 <wire x1="71.12" y1="96.52" x2="83.82" y2="96.52" width="0.1524" layer="91"/>
 </segment>
 </net>
-<net name="N$8" class="0">
+<net name="8" class="0">
 <segment>
 <pinref part="D3" gate="G$1" pin="C"/>
@@
 </segment>
 </net>
-<net name="N$9" class="0">
+<net name="9" class="0">
 <segment>
 <pinref part="R3" gate="G$1" pin="1"/>
-<pinref part="ST6" gate="G$1" pin="1"/>
+<pinref part="LED-3" gate="G$1" pin="1"/>
 <wire x1="106.68" y1="96.52" x2="119.38" y2="96.52" width="0.1524" layer="91"/>
 </segment>
 </net>
-<net name="N$10" class="0">
+<net name="12" class="0">
 <segment>
 <pinref part="R4" gate="G$1" pin="1"/>
-<pinref part="ST8" gate="G$1" pin="1"/>
+<pinref part="LED-4" gate="G$1" pin="1"/>
 <wire x1="106.68" y1="81.28" x2="119.38" y2="81.28" width="0.1524" layer="91"/>
 </segment>
 </net>
-<net name="N$11" class="0">
+<net name="11" class="0">
 <segment>
 <pinref part="D4" gate="G$1" pin="C"/>
@@
 </segment>
 </net>
-<net name="N$12" class="0">
+<net name="10" class="0">
 <segment>
-<pinref part="ST7" gate="G$1" pin="1"/>
+<pinref part="LED+4" gate="G$1" pin="1"/>
 <pinref part="D4" gate="G$1" pin="A"/>
 <wire x1="71.12" y1="81.28" x2="83.82" y2="81.28" width="0.1524" layer="91"/>
 </segment>
 </net>
-<net name="N$13" class="0">
+<net name="13" class="0">
 <segment>
-<pinref part="ST9" gate="G$1" pin="1"/>
+<pinref part="LED+5" gate="G$1" pin="1"/>
 <pinref part="D5" gate="G$1" pin="A"/>
 <wire x1="71.12" y1="66.04" x2="83.82" y2="66.04" width="0.1524" layer="91"/>
 </segment>
 </net>
-<net name="N$14" class="0">
+<net name="14" class="0">
 <segment>
 <pinref part="D5" gate="G$1" pin="C"/>
@@
 </segment>
 </net>
-<net name="N$15" class="0">
+<net name="15" class="0">
 <segment>
 <pinref part="R5" gate="G$1" pin="1"/>
-<pinref part="ST10" gate="G$1" pin="1"/>
+<pinref part="LED-5" gate="G$1" pin="1"/>
 <wire x1="106.68" y1="66.04" x2="119.38" y2="66.04" width="0.1524" layer="91"/>
 </segment>

Commit message: Updated Brd File per Eng Design Rev
Other:
- note added: "LilyPad White LEDs"
- note added: "LilyPad White LEDs are meant to be used with LilyPad Coin Cell Battery (CR2032)"
- note added: "v11"
- note removed: "v02"
Changed lines of the file:
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@@
 <text x="168.402" y="6.604" size="2.54" layer="94">M. West</text>
 <text x="166.116" y="11.43" size="2.54" layer="94">L. Buechley</text>
-<text x="238.76" y="7.62" size="1.778" layer="94">v02</text>
+<text x="238.76" y="7.62" size="1.778" layer="94">v11</text>
+<text x="68.58" y="139.7" size="3.81" layer="97" font="vector">LilyPad White LEDs</text>
+<text x="157.48" y="76.2" size="2.54" layer="97">LilyPad White LEDs are meant
+to be used with LilyPad Coin Cell
+Battery (CR2032)</text>
 </plain>
 <instances>
@@
 </schematic>
 </drawing>
+<compatibility>
+<note version="6.3" minversion="6.2.2" severity="warning">
+Since Version 6.2.2 text objects can contain more than one line,
+which will not be processed correctly with this version.
+</note>
+</compatibility>
 </eagle>
